File: BUG_TRACKING/BUG0004/BUG0004.brd (EAGLE design)
At the start: 12.7 x 12.7 mm, 1 part

Commit message: Created worst case part to test bug
Parts:
- renumbered U$1 to U$1"
Changed lines of the file:
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@@
 </autorouter>
 <elements>
-<element name="U$1" library="test_doublequote" package="TEST" value="TEST&quot;" x="6.35" y="5.08"/>
+<element name="U$1&quot;" library="test_doublequote" package="TEST" value="TEST&quot;" x="6.35" y="5.08">
+<attribute name="TEST" value="&quot;HELLO&quot;" x="6.35" y="5.08" size="1.778" layer="27" display="off"/>
+</element>
 </elements>
 <signals>
